Commit message: multiple visual example

File: FullBody_description/urdf/FullBody.urdf (robot description, URDF)
Before this commit: robot FullBody, 38 links, 37 joints
Links:
- link L_Pelvisv12_1: geometry collision mesh filename=package://meshes/L_Pelvisv12_1.stl scale=0.001 0.001 0.001; visual mesh filename=package://meshes/L_Pelvisv12_1.stl scale=0.001 0.001 0.001
